Commit message: Updated code for final report submission

File: resources/robots/pai_12dof/urdf/pai_12dof copy.urdf (robot description, URDF)
Before this commit: robot pai_12dof_v2_0312, 13 links, 12 joints
Links:
- link l_ankle_roll_link: mass 0.001728932 -> 0.1728932; geometry collision mesh filename=../meshes/l_ankle_roll_link.STL; visual mesh filename=../meshes/l_ankle_roll_link.STL
- link l_calf_link: mass 0.00768122 -> 0.768122
- link l_thigh_link: mass 0.001443603 -> 0.1443603
- link r_ankle_roll_link: mass 0.001728932 -> 0.1728932; geometry collision mesh filename=../meshes/r_ankle_roll_link.STL; visual mesh filename=../meshes/r_ankle_roll_link.STL
- link r_calf_link: mass 0.00768122 -> 0.768122
- link r_thigh_link: mass 0.001443603 -> 0.1443603
